File: labx-final_project/PCB_Design/PCB_Design.kicad_pcb (KiCad board)
At the start: 2 copper layers, 70 x 58 mm, 7 parts, among them M1 Stepper_Motor_x27.168, SW1 SW_SPDT, U1 XIAO ESP32C3

Commit message: add Second PCB Run
Parts:
- BT2: footprint Connector_JST:JST_NV_B02P-NV_1x02_P5.00mm_Vertical -> Connector_JST:JST_PH_B2B-PH-K_1x02_P2.00mm_Vertical
Routing:
- net GND: track 39.5 -> 111.1 mm
- net Net-(Brd1-VCC): track 58.3 -> 78.2 mm
- net Net-(BT2-+): track 12.3 -> 13.4 mm
Other:
- outline, holes or cut-outs redrawn
- board text added: "Wayne's Display Board V2.0"
- board text removed: "Wayne's Display Board V1.0"
