File: labx-final_project/PCB_Design/PCB_Design.kicad_sch (KiCad schematic)
At the start: 7 parts, among them M1 Stepper_Motor_x27.168, SW1 SW_SPDT, U1 XIAO ESP32C3

Commit message: add Second PCB Run
Parts:
- BT2: footprint Connector_JST:JST_NV_B02P-NV_1x02_P5.00mm_Vertical -> Connector_JST:JST_PH_B2B-PH-K_1x02_P2.00mm_Vertical
Changed lines of the file:
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@@
 			)
 		)
-		(property "Footprint" "Connector_JST:JST_NV_B02P-NV_1x02_P5.00mm_Vertical"
+		(property "Footprint" "Connector_JST:JST_PH_B2B-PH-K_1x02_P2.00mm_Vertical"
 			(at 183.896 59.69 90)
 			(effects
